Commit message: Updated till 3A

File: ebot_description/models/ebot/ebot_description_2a.xacro (robot description, xacro)
@@ -25,5 +25,5 @@
         <parent link="ebot_base_link"/>
         <child link="base_footprint"/>
-        <origin xyz="0.0 0.0 0.0" rpy="0.0 0.0 0.0"/>
+        <origin xyz="0.0 0.0 0.220" rpy="0.0 0.0 0.0"/>
     </joint>
     <link name="base_footprint">

Commit message: Updated to requirements for 3B

File: ebot_description/models/ebot/ebot_description_2a.xacro (robot description, xacro)
@@ -25,5 +25,5 @@
         <parent link="ebot_base_link"/>
         <child link="base_footprint"/>
-        <origin xyz="0.0 0.0 0.220" rpy="0.0 0.0 0.0"/>
+        <origin xyz="0.0 0.0 0.0" rpy="0.0 0.0 0.0"/>
     </joint>
     <link name="base_footprint">
